File: Schemetic and Board/WiFi_Tele/fpga_shield.brd (EAGLE design)
At the start: 160 x 100 mm, 32 parts, among them U2 MICROCHIP_MCP1525T-I-TTMICROC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

Commit message: changed mixer
Changed mixer from HMC213B to LT5522 due to stock issues
Parts:
- added C15, C16, C17, C18, C19, C20, C21, C22: 0.01u, rcl:C0805
- added C23, C24, C25, C26: 22pF, rcl:C0805
- added L10, L11, L12, L14, L15, L16, L9, U$6: L2012M, Passives:INDC2518X180
- added R1, R10, R11, R12, R13, R14, R15, R16, R2, R3, R4, R5, R6, R7, R8, R9: 22, rcl:R0805
Connections:
- net N$17 renamed VREF2-5
- removed net N$16: VCO_TUNE.5, VCO_TUNE.7
- removed net N$40: ADC.47, AMP2.44
- removed net N$41: ADC.46, AMP2.43
- new net 1V8: ADC.1, ADC.30, ADC.32, ADC.33, ADC.36, ADC.7
- new net ADC_VCM: ADC.48, R1.1, R2.2, R3.1, R4.2, R5.1, R6.2, R7.1, R8.2
- new net HMCAD1511_CLK_N: ADC.34, SV1.31
- new net HMCAD1511_CLK_P: ADC.35, SV1.32
- new net N$28: AMP2.44, L9.2, R9.1
- new net N$35: AMP2.29, L16.2, R16.1
- new net N$36: ADC.44, C17.2, C24.1, R3.2
- new net N$37: ADC.43, C18.2, C24.2, R4.1
- new net N$38: ADC.41, C19.2, C25.1, R5.2
- new net N$39: ADC.40, C20.2, C25.2, R6.1
- new net N$42: ADC.38, C21.2, C26.1, R7.2
- new net N$43: ADC.37, C22.2, C26.2, R8.1
- new net N$44: ADC.46, C16.2, C23.2, R2.1
- new net N$45: ADC.47, C15.2, C23.1, R1.2
- new net N$46: C15.1, R9.2
- new net N$49: C16.1, R10.2
- new net N$50: C17.1, R11.2
- new net N$51: C18.1, R12.2
- new net N$52: C19.1, R13.2
- new net N$53: C20.1, R14.2
- new net N$54: C21.1, R15.2
- new net N$55: C22.1, R16.2
- new net N$58: ADC.6
- new net N$59: ADC.5
- net GND: now also ADC.29, ADC.31, ADC.39, ADC.42, ADC.45, ADC.49, ADC.8, L10.1, L11.1, L12.1, L14.1, L15.1, L16.1, L9.1, U$6.1, VCO_TUNE.5, VCO_TUNE.7
- net HMCAD1511_CS: now also ADC.2
- net HMCAD1511_D1A_N: now also ADC.10
- net HMCAD1511_D1A_P: now also ADC.9
- net HMCAD1511_D1B_N: now also ADC.12
- net HMCAD1511_D1B_P: now also ADC.11
- net HMCAD1511_D2A_N: now also ADC.14
- net HMCAD1511_D2A_P: now also ADC.13
- net HMCAD1511_D2B_N: now also ADC.16
- net HMCAD1511_D2B_P: now also ADC.15
- net HMCAD1511_D3A_N: now also ADC.22
- net HMCAD1511_D3A_P: now also ADC.21
- net HMCAD1511_D3B_N: now also ADC.24
- net HMCAD1511_D3B_P: now also ADC.23
- net HMCAD1511_D4A_N: now also ADC.26
- net HMCAD1511_D4A_P: now also ADC.25
- net HMCAD1511_D4B_N: now also ADC.28
- net HMCAD1511_D4B_P: now also ADC.27
- net HMCAD1511_FCLK_N: now also ADC.20
- net HMCAD1511_FCLK_P: now also ADC.19
- net HMCAD1511_LCLK_N: now also ADC.18
- net HMCAD1511_LCLK_P: now also ADC.17
- net N$29: now also AMP2.43, L10.2, R10.1; no longer ADC.44, AMP2.39
- net N$30: now also AMP2.39, L11.2, R11.1; no longer ADC.43, AMP2.38
- net N$31: now also AMP2.38, L12.2, R12.1; no longer ADC.41, AMP2.35
- net N$32: now also AMP2.35, L14.2, R13.1; no longer ADC.40, AMP2.34
- net N$33: now also AMP2.34, R14.1, U$6.2; no longer ADC.38, AMP2.30
- net N$34: now also AMP2.30, L15.2, R15.1; no longer ADC.37, AMP2.29
- net SPI_CLK: now also ADC.4
- net SPI_MOSI: now also ADC.3

Commit message: Start FPGA board routing
Routed SMA -> VGA1 matched diff pairs
Parts:
- added C27, C28, C29, C30: 1000uF, rcl:150CLZ-1010
- added C31, C32, C33, C34, C35: 0.1uF, rcl:C0805
- added R17, R18, R19, R20, R21, R22, R23, R24, R25, R26: 100, rcl:R0603
- added SV2, SV3, SV4: (no value), con-lstb:MA05-1
- added VREG1: TLV75718PDBVR, Tl757p:SOT95P240X110-5
- L10, L11, L12, L14, L15, L16, L9, U$6: value L2012M -> 1uH
- moved CH2 143.2 mm to (150.2, 62.4)
- moved CH3 140.7 mm to (150.2, 73.2)
- moved CH1 140.6 mm to (150.2, 52.1)
- moved C3 127.6 mm to (-47.0, -25.4)
- moved AMP_1 98.0 mm to (129.7, 67.5)
- moved CH4 97.4 mm to (150.2, 83.5)
- moved C9 82.5 mm to (86.1, 123.1)
- moved C1 82.5 mm to (83.5, 129.5)
- moved C10 82.5 mm to (78.5, 123.1)
- moved C11 82.5 mm to (65.8, 123.1)
- moved C13 82.5 mm to (95.0, 129.5)
- moved C14 82.5 mm to (88.6, 129.5)
- moved C2 82.5 mm to (72.1, 123.1)
- moved C4 82.5 mm to (81.0, 114.2)
- moved C5 82.5 mm to (73.4, 114.2)
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Connections:
- net N$1 renamed IF1_P
- net N$10 renamed AMP1_OA_N
- net N$11 renamed AMP1_OB_P
- net N$12 renamed AMP1_OB_N
- net N$13 renamed AMP1_OC_P
- net N$14 renamed AMP1_OC_N
- net N$15 renamed AMP1_OD_P
- net N$19 renamed AMP1_OD_N
- net N$2 renamed IF2_P
- net N$26 renamed AMP2_IA_N
- net N$27 renamed AMP2_IA_P
- net N$28 renamed AMP2_OA1_P
- net N$29 renamed AMP2_OA1_N
- net N$3 renamed IF3_P
- net N$30 renamed AMP2_OB1_P
- net N$31 renamed AMP2_OB1_N
- net N$32 renamed AMP2_OC1_P
- net N$33 renamed AMP2_OC1_N
- net N$34 renamed AMP2_OD1_P
- net N$35 renamed AMP2_OD1_N
- net N$36 renamed ADC_IN2_P
- net N$37 renamed ADC_IN2_N
- net N$38 renamed ADC_IN3_P
- net N$39 renamed ADC_IN3_N
- net N$4 renamed IF4_P
- net N$42 renamed ADC_IN4_P
- net N$43 renamed ADC_IN4_N
- net N$44 renamed ADC_IN1_N
- net N$45 renamed ADC_IN1_P
- net N$46 renamed AMP2_OA2_P
- net N$49 renamed AMP2_OA2_N
- net N$5 renamed IF4_N
- net N$50 renamed AMP2_OB2_P
- net N$51 renamed AMP2_OB2_N
- net N$52 renamed AMP2_OC2_P
- net N$53 renamed AMP2_OC2_N
- net N$54 renamed AMP2_OD2_P
- net N$55 renamed AMP2_OD2_N
- net N$6 renamed AMP1_OA_P
- net N$7 renamed IF3_N
- net N$8 renamed IF2_N
- net N$9 renamed IF1_N
- removed net N$20: AMP2.16, C9.2, L7.2, L8.2
- removed net N$21: AMP2.17, C10.2
- removed net N$22: AMP2.12, C8.2
- removed net N$23: AMP2.11, C7.2, L5.2, L6.2
- removed net N$24: AMP2.8, C6.2
- removed net N$25: AMP2.7, C5.2, L3.2, L4.2
- removed net N$58: ADC.6
- removed net N$59: ADC.5
- new net AMP2_IB_N: AMP2.8, C6.2, L4.2
- new net AMP2_IB_P: AMP2.7, C5.2, L3.2
- new net AMP2_IC_N: AMP2.12, C8.2, L6.2
- new net AMP2_IC_P: AMP2.11, C7.2, L5.2
- new net AMP2_ID_N: AMP2.17, C10.2, L8.2
- new net AMP2_ID_P: AMP2.16, C9.2, L7.2
- new net N$17: C27.-, C28.-, C29.-
- net 1V8: now also ADC.5, C30.+, C31.1, C32.1, C33.1, C34.1, C35.1, VREG1.5
- net 5V: now also C27.+, C28.+, C29.+, SV2.4, SV3.4, SV4.4, VREG1.1, VREG1.3
- net GND: now also ADC.6, C30.-, C31.2, C32.2, C33.2, C34.2, C35.2, SV2.1, SV2.3, SV2.5, SV3.1, SV3.3, SV3.5, SV4.1, SV4.3, SV4.5, VREG1.2, VREG1.4
- net HMCAD1511_D1A_N: now also R17.1
- net HMCAD1511_D1A_P: now also R17.2
- net HMCAD1511_D1B_N: now also R18.1
- net HMCAD1511_D1B_P: now also R18.2
- net HMCAD1511_D2A_N: now also R19.1
- net HMCAD1511_D2A_P: now also R19.2
- net HMCAD1511_D2B_N: now also R20.1
- net HMCAD1511_D2B_P: now also R20.2
- net HMCAD1511_D3A_N: now also R23.1
- net HMCAD1511_D3A_P: now also R23.2
- net HMCAD1511_D3B_N: now also R24.1
- net HMCAD1511_D3B_P: now also R24.2
- net HMCAD1511_D4A_N: now also R25.1
- net HMCAD1511_D4A_P: now also R25.2
- net HMCAD1511_D4B_N: now also R26.1
- net HMCAD1511_D4B_P: now also R26.2
- net HMCAD1511_FCLK_N: now also R22.1
- net HMCAD1511_FCLK_P: now also R22.2
- net HMCAD1511_LCLK_N: now also R21.1
- net HMCAD1511_LCLK_P: now also R21.2
- net V_TUNE: now also SV2.2, SV3.2, SV4.2
Routing:
- net IF3_P: track 0.00 -> 20.5 mm
- net IF3_N: track 0.00 -> 20.5 mm
- net IF1_N: track 0.00 -> 19.4 mm
- net IF1_P: track 0.00 -> 19.4 mm
- net IF2_P: track 0.00 -> 19.3 mm
- net IF2_N: track 0.00 -> 19.3 mm
- net IF4_P: track 0.00 -> 19.3 mm
- net IF4_N: track 0.00 -> 19.3 mm

Commit message: completed two VGA routing
Parts:
- removed U$6: 1uH, Passives:INDC2518X180
- added C36, C37, C38, C39: 0.1uF, rcl:C0805
- added L13: 1uH, Passives:INDC2518X180
- added R27, R28: 2000, rcl:R0805
- C10, C3, C4, C5, C6, C7, C8, C9: device rcl:C0805 -> rcl:C0603
- moved SV4 279.1 mm to (123.0, 9.29), turned to 90 degrees
- moved VREG1 277.6 mm to (41.3, 16.5), turned to 180 degrees
- moved C29 271.2 mm to (56.5, 9.16), turned to 90 degrees
- moved SV3 268.0 mm to (114.9, 9.29), turned to 90 degrees
- moved C28 266.4 mm to (69.3, 9.16), turned to 90 degrees
- moved C27 263.1 mm to (82.9, 9.16), turned to 90 degrees
- moved C22 260.8 mm to (54.4, 51.0), turned to 180 degrees
- moved SV2 256.4 mm to (105.8, 9.29), turned to 90 degrees
- moved C21 254.1 mm to (54.4, 48.6), turned to 180 degrees
- moved C20 242.3 mm to (50.5, 42.5), turned to 180 degrees
- moved C19 235.4 mm to (50.4, 39.9), turned to 180 degrees
- moved C18 227.7 mm to (54.4, 33.9), turned to 180 degrees
- moved R16 226.1 mm to (58.9, 51.0), turned to 180 degrees
- moved C17 221.1 mm to (54.4, 31.3), turned to 180 degrees
- moved R15 219.7 mm to (58.9, 48.6), turned to 180 degrees
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Connections:
- removed net N$17: C27.-, C28.-, C29.-
- removed net SPI_MISO: AMP2.45, AMP_1.45
- new net N$1: AMP_1.45, R27.1
- new net N$2: AMP2.45, R28.1
- net 5V: now also C36.1, C37.1, C38.1, C39.1
- net ADC_IN1_N: now also C21.2, C26.1, R7.2; no longer C16.2, C23.2, R2.1
- net ADC_IN1_P: now also C22.2, C26.2, R8.1; no longer C15.2, C23.1, R1.2
- net ADC_IN2_N: now also C19.2, C25.1, R5.2; no longer C18.2, C24.2, R4.1
- net ADC_IN2_P: now also C20.2, C25.2, R6.1; no longer C17.2, C24.1, R3.2
- net ADC_IN3_N: now also C17.2, C24.1, R3.2; no longer C20.2, C25.2, R6.1
- net ADC_IN3_P: now also C18.2, C24.2, R4.1; no longer C19.2, C25.1, R5.2
- net ADC_IN4_N: now also C15.2, C23.1, R1.2; no longer C22.2, C26.2, R8.1
- net ADC_IN4_P: now also C16.2, C23.2, R2.1; no longer C21.2, C26.1, R7.2
- net AMP1_OA_N: now also L2.2
- net AMP1_OA_P: now also L1.2
- net AMP1_OB_N: now also L4.2
- net AMP1_OB_P: now also L3.2
- net AMP1_OC_N: now also L6.2
- net AMP1_OC_P: now also L5.2
- net AMP1_OD_N: now also L8.2
- net AMP1_OD_P: now also L7.2
- net AMP2_IA_N: no longer L2.2
- net AMP2_IA_P: no longer L1.2
- net AMP2_IB_N: no longer L4.2
- net AMP2_IB_P: no longer L3.2
- net AMP2_IC_N: no longer L6.2
- net AMP2_IC_P: no longer L5.2
- net AMP2_ID_N: no longer L8.2
- net AMP2_ID_P: no longer L7.2
- net AMP2_OC1_N: now also L14.2; no longer U$6.2
- net AMP2_OC1_P: now also L13.2; no longer L14.2
- net GND: now also C27.-, C28.-, C29.-, C36.2, C37.2, C38.2, C39.2, L13.1, R27.2, R28.2; no longer U$6.1
- net HMCAD1511_D1A_N: now also SV1.1; no longer SV1.8
- net HMCAD1511_D1A_P: now also SV1.4; no longer SV1.7
- net HMCAD1511_D1B_N: now also SV1.6; no longer SV1.17
- net HMCAD1511_D1B_P: now also SV1.5; no longer SV1.18
- net HMCAD1511_D2A_N: now also SV1.8; no longer SV1.21
- net HMCAD1511_D2A_P: now also SV1.7; no longer SV1.22
- net HMCAD1511_D2B_N: now also SV1.17; no longer SV1.25
- net HMCAD1511_D2B_P: now also SV1.18; no longer SV1.26
- net HMCAD1511_FCLK_N: now also SV1.25; no longer SV1.1
- net HMCAD1511_FCLK_P: now also SV1.26; no longer SV1.4
- net HMCAD1511_LCLK_N: now also SV1.21; no longer SV1.6
- net HMCAD1511_LCLK_P: now also SV1.22; no longer SV1.5
Routing:
- net GND: track 0.00 -> 246.4 mm, vias 0 -> 50
- net SPI_MOSI: track 0.00 -> 201.7 mm, vias 0 -> 3
- net SPI_CLK: track 0.00 -> 193.9 mm, vias 0 -> 3
- net AMP1_CS: track 0.00 -> 145.8 mm, vias 0 -> 1
- net MCP4921_CS: track 0.00 -> 131.4 mm, vias 0 -> 2
- net AMP2_CS: track 0.00 -> 75.8 mm, vias 0 -> 1
- net HMCAD1511_D2B_N: track 0.00 -> 69.2 mm
- net HMCAD1511_FCLK_N: track 0.00 -> 68.6 mm
- net HMCAD1511_D4A_N: track 0.00 -> 67.3 mm
- net HMCAD1511_D3A_N: track 0.00 -> 66.5 mm
- net HMCAD1511_D4B_P: track 0.00 -> 66.4 mm
- net HMCAD1511_D3B_N: track 0.00 -> 66.2 mm
- net HMCAD1511_LCLK_N: track 0.00 -> 66.1 mm
- net HMCAD1511_FCLK_P: track 0.00 -> 65.9 mm
- net HMCAD1511_D4A_P: track 0.00 -> 64.2 mm
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- added copper zone on layer 15, net 1V8
- added copper zone on layer 1, net 5V
- added copper zone on layer 15, net 5V
- added copper zone on layer 1, net ADC_VCM
- added copper zone on layer 15, net ADC_VCM
- added copper zone on layer 1, net GND
- added copper zone on layer 2, net GND
- added copper zone on layer 1, net IF1_N
- added copper zone on layer 1, net IF2_N
- added copper zone on layer 1, net IF3_N
- added copper zone on layer 1, net IF4_N
Other:
- board size 160 x 100 mm -> 131.5 x 55.5 mm
- board text added: "ETH PORT VVV"
- board text added: "^ FPGA ^"

Commit message: board complete and send for manufacturing
Parts:
- removed AMP_1: LMH6522_NJY_54, LMH6522:SQA54A
- removed C10, C3, C4, C5, C6, C7, C8, C9: 0.01uF, rcl:C0603
- removed C36, C37, C38, C39: 0.1uF, rcl:C0805
- removed L1, L2, L3, L4, L5, L6, L7, L8: 1uH, Passives:INDC2518X180
- removed R27: 2000, rcl:R0805
- moved CH1 35.0 mm to (83.2, 24.6)
- moved CH4 35.0 mm to (83.2, 49.5)
- moved CH3 34.0 mm to (92.2, 42.1)
- moved CH2 34.0 mm to (92.2, 32.4)
- moved SV4 25.9 mm to (99.2, 19.5), turned to 180 degrees
- moved C11 12.2 mm to (73.3, 44.1)
- moved SV3 11.5 mm to (103.4, 8.29)
- moved VCO_TUNE 9.00 mm to (88.4, 5.58)
- moved SV2 8.56 mm to (97.3, 8.29)
- moved C1 7.46 mm to (92.5, 9.46), turned to 0 degrees
- moved C2 6.50 mm to (83.6, 11.9)
- moved C27 6.50 mm to (76.4, 9.16)
- moved C28 6.50 mm to (62.8, 9.16)
- moved C29 6.50 mm to (50.0, 9.16)
- moved U2 6.50 mm to (88.5, 11.9)
- renumbered AMP2 to AMP
Connections:
- net AMP2_CS renamed AMP_CS
- removed net AMP1_CS: AMP_1.47, SV1.10
- removed net AMP1_OA_N: AMP_1.43, C4.1, L2.2
- removed net AMP1_OA_P: AMP_1.44, C3.1, L1.2
- removed net AMP1_OB_N: AMP_1.38, C6.1, L4.2
- removed net AMP1_OB_P: AMP_1.39, C5.1, L3.2
- removed net AMP1_OC_N: AMP_1.34, C8.1, L6.2
- removed net AMP1_OC_P: AMP_1.35, C7.1, L5.2
- removed net AMP1_OD_N: AMP_1.29, C10.1, L8.2
- removed net AMP1_OD_P: AMP_1.30, C9.1, L7.2
- removed net AMP2_IA_N: AMP.3, C4.2
- removed net AMP2_IA_P: AMP.2, C3.2
- removed net AMP2_IB_N: AMP.8, C6.2
- removed net AMP2_IB_P: AMP.7, C5.2
- removed net AMP2_IC_N: AMP.12, C8.2
- removed net AMP2_IC_P: AMP.11, C7.2
- removed net AMP2_ID_N: AMP.17, C10.2
- removed net AMP2_ID_P: AMP.16, C9.2
- removed net N$1: AMP_1.45, R27.1
- net 5V: no longer AMP_1.31, AMP_1.33, AMP_1.40, AMP_1.42, AMP_1.5, C36.1, C37.1, C38.1, C39.1
- net GND: no longer AMP_1.1, AMP_1.10, AMP_1.13, AMP_1.14, AMP_1.15, AMP_1.18, AMP_1.19, AMP_1.20, AMP_1.21, AMP_1.22, AMP_1.23, AMP_1.24, AMP_1.25, AMP_1.26, AMP_1.27, AMP_1.28, AMP_1.32, AMP_1.36, AMP_1.37, AMP_1.4, AMP_1.41, AMP_1.49, AMP_1.50, AMP_1.51, AMP_1.52, AMP_1.53, AMP_1.54, AMP_1.55, AMP_1.6, AMP_1.9, C36.2, C37.2, C38.2, C39.2, L1.1, L2.1, L3.1, L4.1, L5.1, L6.1, L7.1, L8.1, R27.2
- net IF1_N: now also AMP.3; no longer AMP_1.3
- net IF1_P: now also AMP.2; no longer AMP_1.2
- net IF2_N: now also AMP.8; no longer AMP_1.8
- net IF2_P: now also AMP.7; no longer AMP_1.7
- net IF3_N: now also AMP.12; no longer AMP_1.12
- net IF3_P: now also AMP.11; no longer AMP_1.11
- net IF4_N: now also AMP.17; no longer AMP_1.17
- net IF4_P: now also AMP.16; no longer AMP_1.16
- net SPI_CLK: no longer AMP_1.48
- net SPI_MOSI: no longer AMP_1.46
Routing:
- net AMP1_CS: track 145.8 -> 0.00 mm, vias 1 -> 0
- net GND: track 246.4 -> 114.3 mm, vias 50 -> 355
- net SPI_MOSI: track 201.7 -> 115.5 mm
- net SPI_CLK: track 193.9 -> 118.0 mm
- net 5V: track 48.8 -> 21.1 mm, vias 29 -> 22
- net AMP1_OC_P: track 27.5 -> 0.00 mm
- net AMP1_OC_N: track 27.5 -> 0.00 mm
- net AMP1_OD_P: track 24.6 -> 0.00 mm
- net AMP1_OD_N: track 24.5 -> 0.00 mm
- net AMP1_OA_P: track 24.0 -> 0.00 mm
- net AMP1_OB_N: track 23.9 -> 0.00 mm
- net AMP1_OB_P: track 23.9 -> 0.00 mm
- net AMP1_OA_N: track 23.8 -> 0.00 mm
- net AMP2_IA_P: track 16.6 -> 0.00 mm
- net AMP2_IA_N: track 16.5 -> 0.00 mm
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Other:
- board size 131.5 x 55.5 mm -> 107 x 55.5 mm
- board text added: "Phased Array WiFi IF ADC"
- board text added: "V1 by Alistair Symonds"

Commit message: Deleted a whole bunch of stuff which shouldn't be in the repo
Parts:
- added R27: 120, rcl:R0402
- added R29, R30: 170, rcl:R0402
- added R31: 100, rcl:R0402
- added SV5: (no value), con-lstb:MA05-1
- R17, R18, R19, R20, R21, R22, R23, R24, R25, R26: device rcl:R0603 -> rcl:R0402
- moved C32 18.4 mm to (30.4, 26.4), turned to 270 degrees
- moved R18 5.35 mm to (7.27, 45.6), turned to 0 degrees
- moved R19 5.02 mm to (7.27, 43.1), turned to 0 degrees
- moved R26 4.95 mm to (7.34, 3.85)
- moved R23 4.90 mm to (7.27, 17.7), turned to 180 degrees
- moved R25 4.60 mm to (7.24, 7.52), turned to 180 degrees
- moved R20 4.49 mm to (7.17, 30.4), turned to 180 degrees
- moved R22 4.49 mm to (7.29, 20.2), turned to 180 degrees
- moved R21 4.46 mm to (7.28, 25.2), turned to 180 degrees
- moved R24 4.44 mm to (7.27, 10.00), turned to 180 degrees
- moved R17 4.28 mm to (7.83, 49.7), turned to 180 degrees
- moved C35 1.12 mm to (28.3, 26.7)
- moved SV4 1.12 mm to (98.7, 18.5)
- moved C34 0.50 mm to (32.5, 26.4)
Connections:
- removed net 5V_GPIO: SV1.12
- removed net N$18: C2.2, U2.1
- new net 3V3: ADC.33, C32.1
- new net C10IO_HMCAD1511_CLK_N: R29.1, SV1.31
- new net C10IO_HMCAD1511_CLK_P: R30.1, SV1.32
- net 1V8: no longer ADC.33, C32.1
- net 5V: now also C2.2, SV1.12, SV5.4, U2.1
- net GND: now also SV5.1, SV5.3, SV5.5
- net HMCAD1511_CLK_N: now also R27.2, R29.2, R31.2; no longer SV1.31
- net HMCAD1511_CLK_P: now also R27.1, R30.2, R31.1; no longer SV1.32
- net V_TUNE: now also SV5.2
Routing:
- net GND: track 114.3 -> 59.3 mm, vias 355 -> 365
- net 1V8: track 66.7 -> 45.9 mm
- net 5V: track 21.1 -> 28.1 mm
- net HMCAD1511_D1B_P: track 48.0 -> 41.4 mm
- net HMCAD1511_D2A_P: track 49.1 -> 42.9 mm
- net HMCAD1511_D3A_N: track 66.5 -> 60.4 mm
- net HMCAD1511_D4A_N: track 67.3 -> 61.6 mm
- net HMCAD1511_D2B_N: track 69.2 -> 63.7 mm
- net HMCAD1511_D3B_N: track 66.2 -> 60.6 mm
- net HMCAD1511_FCLK_N: track 68.6 -> 63.1 mm
- net HMCAD1511_LCLK_N: track 66.1 -> 60.7 mm
- net HMCAD1511_D1A_P: track 38.1 -> 32.8 mm
- net HMCAD1511_CLK_P: track 35.0 -> 29.7 mm
- net HMCAD1511_D4B_P: track 66.4 -> 61.2 mm
- net C10IO_HMCAD1511_CLK_P: track 0.00 -> 4.87 mm
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- added copper zone on layer 1, net NOT_GND
- added copper zone on layer 1, net NO_GND
Other:
- board text added: "5V"
- board text added: "V2 by Alistair Symonds"
- board text added: "V_t"
- board text removed: "V1 by Alistair Symonds"
