File: Schemetic and Board/WiFi_Tele/fpga_shield.sch (EAGLE design)
At the start: 0 parts

Commit message: more stuff
Parts:
- added ADC: HMCAD1511, HMCAD1511:HMCAD1511
- added AMP2, AMP_1: LMH6522_NJY_54, LMH6522:LMH6522_NJY_54
- added C1: 1uF, rcl:C-EUC0805
- added C10, C3, C4, C5, C6, C7, C8, C9: 0.01uF, rcl:C-EUC0805
- added C11, C12, C13, C14, C2: 0.1uF, rcl:C-EUC0805
- added CH1, CH2, CH3, CH4: 5-1814832-1, 5-1814832-1:5-1814832-1
- added L1, L2, L3, L4, L5, L6, L7, L8: 1uH, Passives:L2012M
- added SV1: (no value), con-lsta:FE20-2
- added U2: MICROCHIP_MCP1525T-I-TTMICROCHIP_MCP1525T-I-TT_0_1, MCP1525-TT:MICROCHIP_MCP1525T-I-TTMICROCHIP_MCP1525T-I-TT_0_1
- added VCO_TUNE: MCP4921-E_SN, MCP4921-E_SN:MCP4921-E_SN
Connections:
- new net 3V3_GPIO: SV1.30
- new net 5V: AMP2.5VA+, AMP2.5VB+, AMP2.5VC+, AMP2.5VD+, AMP2.MODE, AMP_1.5VA+, AMP_1.5VB+, AMP_1.5VC+, AMP_1.5VD+, AMP_1.MODE, C11.1, C12.1, C13.1, C14.1, VCO_TUNE.VDD
- new net 5V_GPIO: SV1.12
- new net AMP1_CS: AMP_1.A2/CSB, SV1.10
- new net AMP2_CS: AMP2.A2/CSB, SV1.3
- new net GND: AMP2.55, AMP2.A0, AMP2.B0, AMP2.B1, AMP2.B2, AMP2.B3, AMP2.B4, AMP2.C0, AMP2.C1, AMP2.C2, AMP2.C3, AMP2.C4, AMP2.D0, AMP2.D1, AMP2.D2, AMP2.D3, AMP2.D4, AMP2.ENBA, AMP2.ENBB, AMP2.ENBC, AMP2.ENBD, AMP2.GND, AMP2.GND_2, AMP2.GND_3, AMP2.GND_4, AMP2.GND_5, AMP2.GND_6, AMP2.GND_7, AMP2.GND_8, AMP2.GND_9, AMP_1.55, AMP_1.A0, AMP_1.B0, AMP_1.B1, AMP_1.B2, AMP_1.B3, AMP_1.B4, AMP_1.C0, AMP_1.C1, AMP_1.C2, AMP_1.C3, AMP_1.C4, AMP_1.D0, AMP_1.D1, AMP_1.D2, AMP_1.D3, AMP_1.D4, AMP_1.ENBA, AMP_1.ENBB, AMP_1.ENBC, AMP_1.ENBD, AMP_1.GND, AMP_1.GND_2, AMP_1.GND_3, AMP_1.GND_4, AMP_1.GND_5, AMP_1.GND_6, AMP_1.GND_7, AMP_1.GND_8, AMP_1.GND_9, C1.2, C11.2, C12.2, C13.2, C14.2, C2.1, L1.1, L2.1, L3.1, L4.1, L5.1, L6.1, L7.1, L8.1, SV1.11, SV1.29, U2.VSS
- new net HMCAD1511_CS: SV1.2
- new net HMCAD1511_D1A_N: SV1.8
- new net HMCAD1511_D1A_P: SV1.7
- new net HMCAD1511_D1B_N: SV1.17
- new net HMCAD1511_D1B_P: SV1.18
- new net HMCAD1511_D2A_N: SV1.21
- new net HMCAD1511_D2A_P: SV1.22
- new net HMCAD1511_D2B_N: SV1.25
- new net HMCAD1511_D2B_P: SV1.26
- new net HMCAD1511_D3A_N: SV1.27
- new net HMCAD1511_D3A_P: SV1.28
- new net HMCAD1511_D3B_N: SV1.33
- new net HMCAD1511_D3B_P: SV1.34
- new net HMCAD1511_D4A_N: SV1.35
- new net HMCAD1511_D4A_P: SV1.36
- new net HMCAD1511_D4B_N: SV1.40
- new net HMCAD1511_D4B_P: SV1.37
- new net HMCAD1511_FCLK_N: SV1.1
- new net HMCAD1511_FCLK_P: SV1.4
- new net HMCAD1511_LCLK_N: SV1.6
- new net HMCAD1511_LCLK_P: SV1.5
- new net MCP4921_CS: SV1.9, VCO_TUNE.!CS
- new net N$1: AMP_1.INA+, CH1.1
- new net N$10: AMP_1.OUTA-, C4.1
- new net N$11: AMP_1.OUTB+, C5.1
- new net N$12: AMP_1.OUTB-, C6.1
- new net N$13: AMP_1.OUTC+, C7.1
- new net N$14: AMP_1.OUTC-, C8.1
- new net N$15: AMP_1.OUTD+, C9.1
- new net N$16: VCO_TUNE.!LDAC, VCO_TUNE.VSS
- new net N$17: C1.1, U2.OUT, VCO_TUNE.VREF
- new net N$18: C2.2, U2.IN
- new net N$19: AMP_1.OUTD-, C10.1
- new net N$2: AMP_1.INB+, CH2.1
- new net N$20: AMP2.IND+, C9.2, L7.2, L8.2
- new net N$21: AMP2.IND-, C10.2
- new net N$22: AMP2.INC-, C8.2
- new net N$23: AMP2.INC+, C7.2, L5.2, L6.2
- new net N$24: AMP2.INB-, C6.2
- new net N$25: AMP2.INB+, C5.2, L3.2, L4.2
- new net N$26: AMP2.INA-, C4.2, L2.2
- new net N$27: AMP2.INA+, C3.2, L1.2
- new net N$29: ADC.IP2, AMP2.OUTB+
- new net N$3: AMP_1.INC+, CH3.1
- new net N$30: ADC.IN2, AMP2.OUTB-
- new net N$31: ADC.IP3, AMP2.OUTC+
- new net N$32: ADC.IN3, AMP2.OUTC-
- new net N$33: ADC.IP4, AMP2.OUTD+
- new net N$34: ADC.IN4, AMP2.OUTD-
- new net N$4: AMP_1.IND+, CH4.1
- new net N$40: ADC.IP1, AMP2.OUTA+
- new net N$41: ADC.IN1, AMP2.OUTA-
- new net N$5: AMP_1.IND-, CH4.2
- new net N$6: AMP_1.OUTA+, C3.1
- new net N$7: AMP_1.INC-, CH3.2
- new net N$8: AMP_1.INB-, CH2.2
- new net N$9: AMP_1.INA-, CH1.2
- new net SPI_CLK: AMP2.A1/CLK, AMP_1.A1/CLK, SV1.14, VCO_TUNE.SDI
- new net SPI_MISO: AMP2.A4/SDO, AMP_1.A4/SDO
- new net SPI_MOSI: AMP2.A3/SDI, AMP_1.A3/SDI, SV1.13, VCO_TUNE.SCK
- new net V_TUNE: VCO_TUNE.VOUT

Commit message: changed mixer
Changed mixer from HMC213B to LT5522 due to stock issues
Parts:
- added C15, C16, C17, C18, C19, C20, C21, C22: 0.01u, rcl:C-EUC0805
- added C23, C24, C25, C26: 22pF, rcl:C-EUC0805
- added L10, L11, L12, L14, L15, L16, L9, U$6: L2012M, Passives:L2012M
- added R1, R10, R11, R12, R13, R14, R15, R16, R2, R3, R4, R5, R6, R7, R8, R9: 22, rcl:R-US_R0805
Connections:
- net N$17 renamed VREF2-5
- removed net N$16: VCO_TUNE.!LDAC, VCO_TUNE.VSS
- removed net N$40: ADC.IP1, AMP2.OUTA+
- removed net N$41: ADC.IN1, AMP2.OUTA-
- new net 1V8: ADC.AVDD2, ADC.AVDD_1, ADC.AVDD_2, ADC.DVDD_1, ADC.DVDD_2, ADC.OVDD
- new net ADC_VCM: ADC.VCM, R1.1, R2.2, R3.1, R4.2, R5.1, R6.2, R7.1, R8.2
- new net HMCAD1511_CLK_N: ADC.CLKN, SV1.31
- new net HMCAD1511_CLK_P: ADC.CLKP, SV1.32
- new net N$28: AMP2.OUTA+, L9.2, R9.1
- new net N$35: AMP2.OUTD-, L16.2, R16.1
- new net N$36: ADC.IP2, C17.2, C24.1, R3.2
- new net N$37: ADC.IN2, C18.2, C24.2, R4.1
- new net N$38: ADC.IP3, C19.2, C25.1, R5.2
- new net N$39: ADC.IN3, C20.2, C25.2, R6.1
- new net N$42: ADC.IP4, C21.2, C26.1, R7.2
- new net N$43: ADC.IN4, C22.2, C26.2, R8.1
- new net N$44: ADC.IN1, C16.2, C23.2, R2.1
- new net N$45: ADC.IP1, C15.2, C23.1, R1.2
- new net N$46: C15.1, R9.2
- new net N$49: C16.1, R10.2
- new net N$50: C17.1, R11.2
- new net N$51: C18.1, R12.2
- new net N$52: C19.1, R13.2
- new net N$53: C20.1, R14.2
- new net N$54: C21.1, R15.2
- new net N$55: C22.1, R16.2
- new net N$58: ADC.PD
- new net N$59: ADC.RESETN
- net GND: now also ADC.AVSS2, ADC.AVSS_1, ADC.AVSS_2, ADC.AVSS_3, ADC.DVSS_1, ADC.DVSS_2, ADC.EXPOSED_PAD, L10.1, L11.1, L12.1, L14.1, L15.1, L16.1, L9.1, U$6.1, VCO_TUNE.!LDAC, VCO_TUNE.VSS
- net HMCAD1511_CS: now also ADC.CSN
- net HMCAD1511_D1A_N: now also ADC.DN1A
- net HMCAD1511_D1A_P: now also ADC.DP1A
- net HMCAD1511_D1B_N: now also ADC.DN1B
- net HMCAD1511_D1B_P: now also ADC.DP1B
- net HMCAD1511_D2A_N: now also ADC.DN2A
- net HMCAD1511_D2A_P: now also ADC.DP2A
- net HMCAD1511_D2B_N: now also ADC.DN2B
- net HMCAD1511_D2B_P: now also ADC.DP2B
- net HMCAD1511_D3A_N: now also ADC.DN3A
- net HMCAD1511_D3A_P: now also ADC.DP3A
- net HMCAD1511_D3B_N: now also ADC.DN3B
- net HMCAD1511_D3B_P: now also ADC.DP3B
- net HMCAD1511_D4A_N: now also ADC.DN4A
- net HMCAD1511_D4A_P: now also ADC.DP4A
- net HMCAD1511_D4B_N: now also ADC.DN4B
- net HMCAD1511_D4B_P: now also ADC.DP4B
- net HMCAD1511_FCLK_N: now also ADC.FCLKN
- net HMCAD1511_FCLK_P: now also ADC.FCLKP
- net HMCAD1511_LCLK_N: now also ADC.LCLKN
- net HMCAD1511_LCLK_P: now also ADC.LCLKP
- net N$29: now also AMP2.OUTA-, L10.2, R10.1; no longer ADC.IP2, AMP2.OUTB+
- net N$30: now also AMP2.OUTB+, L11.2, R11.1; no longer ADC.IN2, AMP2.OUTB-
- net N$31: now also AMP2.OUTB-, L12.2, R12.1; no longer ADC.IP3, AMP2.OUTC+
- net N$32: now also AMP2.OUTC+, L14.2, R13.1; no longer ADC.IN3, AMP2.OUTC-
- net N$33: now also AMP2.OUTC-, R14.1, U$6.2; no longer ADC.IP4, AMP2.OUTD+
- net N$34: now also AMP2.OUTD+, L15.2, R15.1; no longer ADC.IN4, AMP2.OUTD-
- net SPI_CLK: now also ADC.SCLK
- net SPI_MOSI: now also ADC.SDATA
Other:
- moved on the sheet: ADC

Commit message: Start FPGA board routing
Routed SMA -> VGA1 matched diff pairs
Parts:
- added C27, C28, C29, C30: 1000uF, rcl:CPOL-US150CLZ-1010
- added C31, C32, C33, C34, C35: 0.1uF, rcl:C-EUC0805
- added R17, R18, R19, R20, R21, R22, R23, R24, R25, R26: 100, rcl:R-US_R0603
- added SV2, SV3, SV4: (no value), con-lstb:MA05-1
- added VREG1: TLV75718PDBVR, Tl757p:TLV75718PDBVR
- L10, L11, L12, L14, L15, L16, L9, U$6: value L2012M -> 1uH
Connections:
- net N$1 renamed IF1_P
- net N$10 renamed AMP1_OA_N
- net N$11 renamed AMP1_OB_P
- net N$12 renamed AMP1_OB_N
- net N$13 renamed AMP1_OC_P
- net N$14 renamed AMP1_OC_N
- net N$15 renamed AMP1_OD_P
- net N$19 renamed AMP1_OD_N
- net N$2 renamed IF2_P
- net N$26 renamed AMP2_IA_N
- net N$27 renamed AMP2_IA_P
- net N$28 renamed AMP2_OA1_P
- net N$29 renamed AMP2_OA1_N
- net N$3 renamed IF3_P
- net N$30 renamed AMP2_OB1_P
- net N$31 renamed AMP2_OB1_N
- net N$32 renamed AMP2_OC1_P
- net N$33 renamed AMP2_OC1_N
- net N$34 renamed AMP2_OD1_P
- net N$35 renamed AMP2_OD1_N
- net N$36 renamed ADC_IN2_P
- net N$37 renamed ADC_IN2_N
- net N$38 renamed ADC_IN3_P
- net N$39 renamed ADC_IN3_N
- net N$4 renamed IF4_P
- net N$42 renamed ADC_IN4_P
- net N$43 renamed ADC_IN4_N
- net N$44 renamed ADC_IN1_N
- net N$45 renamed ADC_IN1_P
- net N$46 renamed AMP2_OA2_P
- net N$49 renamed AMP2_OA2_N
- net N$5 renamed IF4_N
- net N$50 renamed AMP2_OB2_P
- net N$51 renamed AMP2_OB2_N
- net N$52 renamed AMP2_OC2_P
- net N$53 renamed AMP2_OC2_N
- net N$54 renamed AMP2_OD2_P
- net N$55 renamed AMP2_OD2_N
- net N$6 renamed AMP1_OA_P
- net N$7 renamed IF3_N
- net N$8 renamed IF2_N
- net N$9 renamed IF1_N
- removed net N$20: AMP2.IND+, C9.2, L7.2, L8.2
- removed net N$21: AMP2.IND-, C10.2
- removed net N$22: AMP2.INC-, C8.2
- removed net N$23: AMP2.INC+, C7.2, L5.2, L6.2
- removed net N$24: AMP2.INB-, C6.2
- removed net N$25: AMP2.INB+, C5.2, L3.2, L4.2
- removed net N$58: ADC.PD
- removed net N$59: ADC.RESETN
- new net AMP2_IB_N: AMP2.INB-, C6.2, L4.2
- new net AMP2_IB_P: AMP2.INB+, C5.2, L3.2
- new net AMP2_IC_N: AMP2.INC-, C8.2, L6.2
- new net AMP2_IC_P: AMP2.INC+, C7.2, L5.2
- new net AMP2_ID_N: AMP2.IND-, C10.2, L8.2
- new net AMP2_ID_P: AMP2.IND+, C9.2, L7.2
- new net N$17: C27.-, C28.-, C29.-
- net 1V8: now also ADC.RESETN, C30.+, C31.1, C32.1, C33.1, C34.1, C35.1, VREG1.OUT
- net 5V: now also C27.+, C28.+, C29.+, SV2.4, SV3.4, SV4.4, VREG1.EN, VREG1.IN
- net GND: now also ADC.PD, C30.-, C31.2, C32.2, C33.2, C34.2, C35.2, SV2.1, SV2.3, SV2.5, SV3.1, SV3.3, SV3.5, SV4.1, SV4.3, SV4.5, VREG1.GND, VREG1.NC
- net HMCAD1511_D1A_N: now also R17.1
- net HMCAD1511_D1A_P: now also R17.2
- net HMCAD1511_D1B_N: now also R18.1
- net HMCAD1511_D1B_P: now also R18.2
- net HMCAD1511_D2A_N: now also R19.1
- net HMCAD1511_D2A_P: now also R19.2
- net HMCAD1511_D2B_N: now also R20.1
- net HMCAD1511_D2B_P: now also R20.2
- net HMCAD1511_D3A_N: now also R23.1
- net HMCAD1511_D3A_P: now also R23.2
- net HMCAD1511_D3B_N: now also R24.1
- net HMCAD1511_D3B_P: now also R24.2
- net HMCAD1511_D4A_N: now also R25.1
- net HMCAD1511_D4A_P: now also R25.2
- net HMCAD1511_D4B_N: now also R26.1
- net HMCAD1511_D4B_P: now also R26.2
- net HMCAD1511_FCLK_N: now also R22.1
- net HMCAD1511_FCLK_P: now also R22.2
- net HMCAD1511_LCLK_N: now also R21.1
- net HMCAD1511_LCLK_P: now also R21.2
- net V_TUNE: now also SV2.2, SV3.2, SV4.2
Other:
- moved on the sheet: R10, R11, R12, R13, R14, R15, R16, R9

Commit message: completed two VGA routing
Parts:
- removed U$6: 1uH, Passives:L2012M
- added C36, C37, C38, C39: 0.1uF, rcl:C-EUC0805
- added L13: 1uH, Passives:L2012M
- added R27, R28: 2000, rcl:R-US_R0805
- C10, C3, C4, C5, C6, C7, C8, C9: device rcl:C-EUC0805 -> rcl:C-EUC0603
Connections:
- removed net N$17: C27.-, C28.-, C29.-
- removed net SPI_MISO: AMP2.A4/SDO, AMP_1.A4/SDO
- new net N$1: AMP_1.A4/SDO, R27.1
- new net N$2: AMP2.A4/SDO, R28.1
- net 5V: now also C36.1, C37.1, C38.1, C39.1
- net ADC_IN1_N: now also C21.2, C26.1, R7.2; no longer C16.2, C23.2, R2.1
- net ADC_IN1_P: now also C22.2, C26.2, R8.1; no longer C15.2, C23.1, R1.2
- net ADC_IN2_N: now also C19.2, C25.1, R5.2; no longer C18.2, C24.2, R4.1
- net ADC_IN2_P: now also C20.2, C25.2, R6.1; no longer C17.2, C24.1, R3.2
- net ADC_IN3_N: now also C17.2, C24.1, R3.2; no longer C20.2, C25.2, R6.1
- net ADC_IN3_P: now also C18.2, C24.2, R4.1; no longer C19.2, C25.1, R5.2
- net ADC_IN4_N: now also C15.2, C23.1, R1.2; no longer C22.2, C26.2, R8.1
- net ADC_IN4_P: now also C16.2, C23.2, R2.1; no longer C21.2, C26.1, R7.2
- net AMP1_OA_N: now also L2.2
- net AMP1_OA_P: now also L1.2
- net AMP1_OB_N: now also L4.2
- net AMP1_OB_P: now also L3.2
- net AMP1_OC_N: now also L6.2
- net AMP1_OC_P: now also L5.2
- net AMP1_OD_N: now also L8.2
- net AMP1_OD_P: now also L7.2
- net AMP2_IA_N: no longer L2.2
- net AMP2_IA_P: no longer L1.2
- net AMP2_IB_N: no longer L4.2
- net AMP2_IB_P: no longer L3.2
- net AMP2_IC_N: no longer L6.2
- net AMP2_IC_P: no longer L5.2
- net AMP2_ID_N: no longer L8.2
- net AMP2_ID_P: no longer L7.2
- net AMP2_OC1_N: now also L14.2; no longer U$6.2
- net AMP2_OC1_P: now also L13.2; no longer L14.2
- net GND: now also C27.-, C28.-, C29.-, C36.2, C37.2, C38.2, C39.2, L13.1, R27.2, R28.2; no longer U$6.1
- net HMCAD1511_D1A_N: now also SV1.1; no longer SV1.8
- net HMCAD1511_D1A_P: now also SV1.4; no longer SV1.7
- net HMCAD1511_D1B_N: now also SV1.6; no longer SV1.17
- net HMCAD1511_D1B_P: now also SV1.5; no longer SV1.18
- net HMCAD1511_D2A_N: now also SV1.8; no longer SV1.21
- net HMCAD1511_D2A_P: now also SV1.7; no longer SV1.22
- net HMCAD1511_D2B_N: now also SV1.17; no longer SV1.25
- net HMCAD1511_D2B_P: now also SV1.18; no longer SV1.26
- net HMCAD1511_FCLK_N: now also SV1.25; no longer SV1.1
- net HMCAD1511_FCLK_P: now also SV1.26; no longer SV1.4
- net HMCAD1511_LCLK_N: now also SV1.21; no longer SV1.6
- net HMCAD1511_LCLK_P: now also SV1.22; no longer SV1.5
Other:
- note added: "Input channels connected to ADC inreverse order to allow easier routing"
- moved on the sheet: ADC, C10, C3, C31, C32, C33, C34, C35, C4, C5, C6, C7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

Commit message: board complete and send for manufacturing
Parts:
- removed AMP_1: LMH6522_NJY_54, LMH6522:LMH6522_NJY_54
- removed C10, C3, C4, C5, C6, C7, C8, C9: 0.01uF, rcl:C-EUC0603
- removed C36, C37, C38, C39: 0.1uF, rcl:C-EUC0805
- removed L1, L2, L3, L4, L5, L6, L7, L8: 1uH, Passives:L2012M
- removed R27: 2000, rcl:R-US_R0805
- renumbered AMP2 to AMP
Connections:
- net AMP2_CS renamed AMP_CS
- removed net AMP1_CS: AMP_1.A2/CSB, SV1.10
- removed net AMP1_OA_N: AMP_1.OUTA-, C4.1, L2.2
- removed net AMP1_OA_P: AMP_1.OUTA+, C3.1, L1.2
- removed net AMP1_OB_N: AMP_1.OUTB-, C6.1, L4.2
- removed net AMP1_OB_P: AMP_1.OUTB+, C5.1, L3.2
- removed net AMP1_OC_N: AMP_1.OUTC-, C8.1, L6.2
- removed net AMP1_OC_P: AMP_1.OUTC+, C7.1, L5.2
- removed net AMP1_OD_N: AMP_1.OUTD-, C10.1, L8.2
- removed net AMP1_OD_P: AMP_1.OUTD+, C9.1, L7.2
- removed net AMP2_IA_N: AMP.INA-, C4.2
- removed net AMP2_IA_P: AMP.INA+, C3.2
- removed net AMP2_IB_N: AMP.INB-, C6.2
- removed net AMP2_IB_P: AMP.INB+, C5.2
- removed net AMP2_IC_N: AMP.INC-, C8.2
- removed net AMP2_IC_P: AMP.INC+, C7.2
- removed net AMP2_ID_N: AMP.IND-, C10.2
- removed net AMP2_ID_P: AMP.IND+, C9.2
- removed net N$1: AMP_1.A4/SDO, R27.1
- net 5V: no longer AMP_1.5VA+, AMP_1.5VB+, AMP_1.5VC+, AMP_1.5VD+, AMP_1.MODE, C36.1, C37.1, C38.1, C39.1
- net GND: no longer AMP_1.55, AMP_1.A0, AMP_1.B0, AMP_1.B1, AMP_1.B2, AMP_1.B3, AMP_1.B4, AMP_1.C0, AMP_1.C1, AMP_1.C2, AMP_1.C3, AMP_1.C4, AMP_1.D0, AMP_1.D1, AMP_1.D2, AMP_1.D3, AMP_1.D4, AMP_1.ENBA, AMP_1.ENBB, AMP_1.ENBC, AMP_1.ENBD, AMP_1.GND, AMP_1.GND_2, AMP_1.GND_3, AMP_1.GND_4, AMP_1.GND_5, AMP_1.GND_6, AMP_1.GND_7, AMP_1.GND_8, AMP_1.GND_9, C36.2, C37.2, C38.2, C39.2, L1.1, L2.1, L3.1, L4.1, L5.1, L6.1, L7.1, L8.1, R27.2
- net IF1_N: now also AMP.INA-; no longer AMP_1.INA-
- net IF1_P: now also AMP.INA+; no longer AMP_1.INA+
- net IF2_N: now also AMP.INB-; no longer AMP_1.INB-
- net IF2_P: now also AMP.INB+; no longer AMP_1.INB+
- net IF3_N: now also AMP.INC-; no longer AMP_1.INC-
- net IF3_P: now also AMP.INC+; no longer AMP_1.INC+
- net IF4_N: now also AMP.IND-; no longer AMP_1.IND-
- net IF4_P: now also AMP.IND+; no longer AMP_1.IND+
- net SPI_CLK: no longer AMP_1.A1/CLK
- net SPI_MOSI: no longer AMP_1.A3/SDI
Other:
- moved on the sheet: CH1, CH2, CH3, CH4

Commit message: Deleted a whole bunch of stuff which shouldn't be in the repo
Parts:
- added R27: 120, rcl:R-US_R0402
- added R29, R30: 170, rcl:R-US_R0402
- added R31: 100, rcl:R-US_R0402
- added SV5: (no value), con-lstb:MA05-1
- R17, R18, R19, R20, R21, R22, R23, R24, R25, R26: device rcl:R-US_R0603 -> rcl:R-US_R0402
Connections:
- removed net 5V_GPIO: SV1.12
- removed net N$18: C2.2, U2.IN
- new net 3V3: ADC.OVDD, C32.1
- new net C10IO_HMCAD1511_CLK_N: R29.1, SV1.31
- new net C10IO_HMCAD1511_CLK_P: R30.1, SV1.32
- net 1V8: no longer ADC.OVDD, C32.1
- net 5V: now also C2.2, SV1.12, SV5.4, U2.IN
- net GND: now also SV5.1, SV5.3, SV5.5
- net HMCAD1511_CLK_N: now also R27.2, R29.2, R31.2; no longer SV1.31
- net HMCAD1511_CLK_P: now also R27.1, R30.2, R31.1; no longer SV1.32
- net V_TUNE: now also SV5.2
Other:
- moved on the sheet: C31
